File: kicad/control.kicad_sch (KiCad schematic)
At the start: 14 parts, among them U10 74LS08, U11 74LS138, U2 74LS112, U8 74LS00, U9 74LS00

Commit message: pcb: move around stuff to make pcb smaller
Parts:
- removed R7: 4K7, Resistor_THT:R_Axial_DIN0207_L6.3mm_D2.5mm_P10.16mm_Horizontal, symbol Device:R
Connections:
- net at R6.1, U2.3 (J): now also U2.4 (~{S})
Other:
- moved on the sheet: R6
Changed lines of the file:
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@@
 	)
 	(junction
+		(at 128.27 35.56)
+		(diameter 0)
+		(color 0 0 0 0)
+	)
+	(junction
 		(at 46.99 129.54)
 		(diameter 0)
@@
 	(wire
 		(pts
+			(xy 128.27 31.75) (xy 128.27 35.56)
+		)
+		(stroke
+			(width 0)
+			(type default)
+		)
+	)
+	(wire
+		(pts
 			(xy 189.23 135.89) (xy 184.15 135.89)
 		)
@@
 	(wire
 		(pts
-			(xy 127 35.56) (xy 127 41.91)
+			(xy 38.1 54.61) (xy 45.72 54.61)
 		)
 		(stroke
@@
 	(wire
 		(pts
-			(xy 38.1 54.61) (xy 45.72 54.61)
+			(xy 46.99 100.33) (xy 46.99 97.79)
 		)
 		(stroke
@@
 	(wire
 		(pts
-			(xy 46.99 100.33) (xy 46.99 97.79)
+			(xy 142.24 110.49) (xy 161.29 110.49)
 		)
 		(stroke
@@
 	(wire
 		(pts
-			(xy 142.24 110.49) (xy 161.29 110.49)
+			(xy 128.27 35.56) (xy 138.43 35.56)
 		)
 		(stroke
@@
 	(wire
 		(pts
+			(xy 128.27 35.56) (xy 128.27 41.91)
+		)
+		(stroke
+			(width 0)
+			(type default)
+		)
+	)
+	(wire
+		(pts
 			(xy 102.87 93.98) (xy 105.41 93.98)
 		)
@@
 	(wire
 		(pts
-			(xy 138.43 26.67) (xy 138.43 27.94)
-		)
-		(stroke
-			(width 0)
-			(type default)
-		)
-	)
-	(wire
-		(pts
 			(xy 49.53 127) (xy 46.99 127)
 		)
@@
 	(wire
 		(pts
-			(xy 130.81 41.91) (xy 127 41.91)
+			(xy 130.81 41.91) (xy 128.27 41.91)
 		)
 		(stroke
@@
 	(symbol
 		(lib_id "Device:R")
-		(at 127 31.75 0)
+		(at 128.27 27.94 0)
 		(mirror x)
 		(unit 1)
@@
 		(dnp no)
 		(property "Reference" "R6"
-			(at 124.46 30.4799 0)
+			(at 125.73 26.6699 0)
 			(effects
 				(font
@@
 		)
 		(property "Value" "4K7"
-			(at 124.46 33.0199 0)
+			(at 125.73 29.2099 0)
 			(effects
 				(font
@@
 		)
 		(property "Footprint" "Resistor_THT:R_Axial_DIN0207_L6.3mm_D2.5mm_P10.16mm_Horizontal"
-			(at 125.222 31.75 90)
+			(at 126.492 27.94 90)
 			(effects
 				(font
@@
 		)
 		(property "Datasheet" "~"
-			(at 127 31.75 0)
+			(at 128.27 27.94 0)
 			(effects
 				(font
@@
 		)
 		(property "Description" "Resistor"
-			(at 127 31.75 0)
+			(at 128.27 27.94 0)
 			(effects
 				(font
@@
 	(symbol
 		(lib_id "power:VCC")
-		(at 138.43 26.67 0)
-		(unit 1)
-		(exclude_from_sim no)
-		(in_bom yes)
-		(on_board yes)
-		(dnp no)
-		(fields_autoplaced yes)
-		(property "Reference" "#PWR019"
-			(at 138.43 30.48 0)
-			(effects
-				(font
-					(size 1.27 1.27)
-				)
-				(hide yes)
-			)
-		)
-		(property "Value" "VCC"
-			(at 138.43 21.59 0)
-			(effects
-				(font
-					(size 1.27 1.27)
-				)
-			)
-		)
-		(property "Footprint" ""
-			(at 138.43 26.67 0)
-			(effects
-				(font
-					(size 1.27 1.27)
-				)
-				(hide yes)
-			)
-		)
-		(property "Datasheet" ""
-			(at 138.43 26.67 0)
-			(effects
-				(font
-					(size 1.27 1.27)
-				)
-				(hide yes)
-			)
-		)
-		(property "Description" "Power symbol creates a global label with name \"VCC\""
-			(at 138.43 26.67 0)
-			(effects
-				(font
-					(size 1.27 1.27)
-				)
-				(hide yes)
-			)
-		)
-		(pin "1"
-		)
-		(instances
-			(project "6502atty"
-				(path "/f612fa92-d5fa-4cb5-a666-c1c24e7cbb30/97889d46-05ef-4a27-a7eb-55210d62cf31"
-					(reference "#PWR019")
-					(unit 1)
-				)
-			)
-		)
-	)
-	(symbol
-		(lib_id "power:VCC")
 		(at 154.94 50.8 0)
 		(unit 1)
@@
 	)
 	(symbol
-		(lib_id "Device:R")
-		(at 138.43 31.75 0)
-		(mirror x)
-		(unit 1)
-		(exclude_from_sim no)
-		(in_bom yes)
-		(on_board yes)
-		(dnp no)
-		(property "Reference" "R7"
-			(at 135.89 30.4799 0)
-			(effects
-				(font
-					(size 1.27 1.27)
-				)
-				(justify right)
-			)
-		)
-		(property "Value" "4K7"
-			(at 135.89 33.0199 0)
-			(effects
-				(font
-					(size 1.27 1.27)
-				)
-				(justify right)
-			)
-		)
-		(property "Footprint" "Resistor_THT:R_Axial_DIN0207_L6.3mm_D2.5mm_P10.16mm_Horizontal"
-			(at 136.652 31.75 90)
-			(effects
-				(font
-					(size 1.27 1.27)
-				)
-				(hide yes)
-			)
-		)
-		(property "Datasheet" "~"
-			(at 138.43 31.75 0)
-			(effects
-				(font
-					(size 1.27 1.27)
-				)
-				(hide yes)
-			)
-		)
-		(property "Description" "Resistor"
-			(at 138.43 31.75 0)
-			(effects
-				(font
-					(size 1.27 1.27)
-				)
-				(hide yes)
-			)
-		)
-		(pin "2"
-		)
-		(pin "1"
-		)
-		(instances
-			(project "6502atty"
-				(path "/f612fa92-d5fa-4cb5-a666-c1c24e7cbb30/97889d46-05ef-4a27-a7eb-55210d62cf31"
-					(reference "R7")
-					(unit 1)
-				)
-			)
-		)
-	)
-	(symbol
 		(lib_id "power:GND")
 		(at 71.12 176.53 0)
@@
 	(symbol
 		(lib_id "power:VCC")
-		(at 127 27.94 0)
+		(at 128.27 24.13 0)
 		(unit 1)
 		(exclude_from_sim no)
@@
 		(fields_autoplaced yes)
 		(property "Reference" "#PWR048"
-			(at 127 31.75 0)
+			(at 128.27 27.94 0)
 			(effects
 				(font
@@
 		)
 		(property "Value" "VCC"
-			(at 127 22.86 0)
+			(at 128.27 19.05 0)
 			(effects
 				(font
@@
 		)
 		(property "Footprint" ""
-			(at 127 27.94 0)
+			(at 128.27 24.13 0)
 			(effects
 				(font
@@
 		)
 		(property "Datasheet" ""
-			(at 127 27.94 0)
+			(at 128.27 24.13 0)
 			(effects
 				(font
@@
 		)
 		(property "Description" "Power symbol creates a global label with name \"VCC\""
-			(at 127 27.94 0)
+			(at 128.27 24.13 0)
 			(effects
 				(font

Commit message: pcb: minor schematic updates
Parts:
- R24: value 1K -> 560R
Other:
- note added: "R24 either low-ohm or wire-link"
- moved on the sheet: R24, R8, U2B
Changed lines of the file:
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@@
 		(comment 1 "© 2025 Ben Dooks")
 	)
+	(text "R24 either low-ohm or wire-link"
+		(exclude_from_sim no)
+		(at 190.5 70.104 0)
+		(effects
+			(font
+				(size 1.27 1.27)
+			)
+		)
+	)
 	(text "ATMega select (ROM or IO)"
 		(exclude_from_sim no)
@@
 	)
 	(junction
-		(at 154.94 59.69)
+		(at 152.4 66.04)
 		(diameter 0)
 		(color 0 0 0 0)
@@
 	(wire
 		(pts
-			(xy 186.69 59.69) (xy 198.12 59.69)
+			(xy 184.15 66.04) (xy 195.58 66.04)
 		)
 		(stroke
@@
 	(wire
 		(pts
-			(xy 158.75 64.77) (xy 154.94 64.77)
+			(xy 156.21 71.12) (xy 152.4 71.12)
 		)
 		(stroke
@@
 	(wire
 		(pts
-			(xy 166.37 69.85) (xy 166.37 74.93)
+			(xy 163.83 76.2) (xy 163.83 81.28)
 		)
 		(stroke
@@
 	(wire
 		(pts
-			(xy 149.86 74.93) (xy 166.37 74.93)
+			(xy 147.32 81.28) (xy 163.83 81.28)
 		)
 		(stroke
@@
 	(wire
 		(pts
-			(xy 173.99 59.69) (xy 179.07 59.69)
+			(xy 171.45 66.04) (xy 176.53 66.04)
 		)
 		(stroke
@@
 	(wire
 		(pts
-			(xy 140.97 62.23) (xy 158.75 62.23)
+			(xy 138.43 68.58) (xy 156.21 68.58)
 		)
 		(stroke
@@
 	(wire
 		(pts
-			(xy 154.94 64.77) (xy 154.94 59.69)
+			(xy 152.4 71.12) (xy 152.4 66.04)
 		)
 		(stroke
@@
 	(wire
 		(pts
-			(xy 148.59 43.18) (xy 148.59 46.99)
-		)
-		(stroke
-			(width 0)
-			(type default)
-		)
-	)
-	(wire
-		(pts
 			(xy 123.19 113.03) (xy 127 113.03)
 		)
@@
 	(wire
 		(pts
-			(xy 146.05 46.99) (xy 148.59 46.99)
+			(xy 146.05 46.99) (xy 163.83 46.99)
 		)
 		(stroke
@@
 	(wire
 		(pts
-			(xy 154.94 58.42) (xy 154.94 59.69)
+			(xy 152.4 57.15) (xy 152.4 54.61)
+		)
+		(stroke
+			(width 0)
+			(type default)
+		)
+	)
+	(wire
+		(pts
+			(xy 152.4 64.77) (xy 152.4 66.04)
 		)
 		(stroke
@@
 	(wire
 		(pts
-			(xy 166.37 43.18) (xy 166.37 54.61)
+			(xy 163.83 46.99) (xy 163.83 60.96)
 		)
 		(stroke
@@
 	(wire
 		(pts
-			(xy 148.59 43.18) (xy 166.37 43.18)
-		)
-		(stroke
-			(width 0)
-			(type default)
-		)
-	)
-	(wire
-		(pts
 			(xy 256.54 130.81) (xy 256.54 135.89)
 		)
@@
 	(wire
 		(pts
-			(xy 154.94 59.69) (xy 158.75 59.69)
+			(xy 152.4 66.04) (xy 156.21 66.04)
 		)
 		(stroke
@@
 	)
 	(label "CPU_~{RESET}"
-		(at 149.86 74.93 0)
+		(at 149.86 81.28 0)
 		(effects
 			(font
@@
 	)
 	(label "CPU_CLK"
-		(at 198.12 59.69 180)
+		(at 195.58 66.04 180)
 		(effects
 			(font
@@
 	)
 	(label "PWM_CLK"
-		(at 140.97 62.23 0)
+		(at 138.43 68.58 0)
 		(effects
 			(font
@@
 	)
 	(label "~{CPU_STOP}"
-		(at 148.59 43.18 0)
+		(at 152.4 46.99 0)
 		(effects
 			(font
@@
 	(hierarchical_label "PWM_CLK"
 		(shape output)
-		(at 140.97 62.23 180)
+		(at 138.43 68.58 180)
 		(effects
 			(font
@@
 	(hierarchical_label "CPU_~{RESET}"
 		(shape input)
-		(at 149.86 74.93 180)
+		(at 147.32 81.28 180)
 		(effects
 			(font
@@
 	(hierarchical_label "CPU_CLK"
 		(shape input)
-		(at 198.12 59.69 0)
+		(at 195.58 66.04 0)
 		(effects
 			(font
@@
 	(symbol
 		(lib_id "74xx:74LS112")
-		(at 166.37 62.23 0)
+		(at 163.83 68.58 0)
 		(unit 2)
 		(exclude_from_sim no)
@@
 		(fields_autoplaced yes)
 		(property "Reference" "U2"
-			(at 168.5133 52.07 0)
+			(at 165.9733 58.42 0)
 			(effects
 				(font
@@
 		)
 		(property "Value" "74LS112"
-			(at 168.5133 54.61 0)
+			(at 165.9733 60.96 0)
 			(effects
 				(font
@@
 		)
 		(property "Footprint" "Package_DIP:DIP-16_W7.62mm"
-			(at 166.37 62.23 0)
+			(at 163.83 68.58 0)
 			(effects
 				(font
@@
 		)
 		(property "Datasheet" "http://www.ti.com/lit/gpn/sn74LS112"
-			(at 166.37 62.23 0)
+			(at 163.83 68.58 0)
 			(effects
 				(font
@@
 		)
 		(property "Description" "dual JK Flip-Flop, Set & Reset"
-			(at 166.37 62.23 0)
+			(at 163.83 68.58 0)
 			(effects
 				(font
@@
 	(symbol
 		(lib_id "Device:R")
-		(at 182.88 59.69 270)
+		(at 180.34 66.04 270)
 		(unit 1)
 		(exclude_from_sim no)
@@
 		(fields_autoplaced yes)
 		(property "Reference" "R24"
-			(at 182.88 53.34 90)
+			(at 180.34 60.8795 90)
 			(effects
 				(font
@@
 			)
 		)
-		(property "Value" "1K"
-			(at 182.88 55.88 90)
+		(property "Value" "560R"
+			(at 180.34 63.3038 90)
 			(effects
 				(font
@@
 		)
 		(property "Footprint" "Resistor_THT:R_Axial_DIN0207_L6.3mm_D2.5mm_P10.16mm_Horizontal"
-			(at 182.88 57.912 90)
+			(at 180.34 64.262 90)
 			(effects
 				(font
@@
 		)
 		(property "Datasheet" "~"
-			(at 182.88 59.69 0)
+			(at 180.34 66.04 0)
 			(effects
 				(font
@@
 		)
 		(property "Description" "Resistor"
-			(at 182.88 59.69 0)
+			(at 180.34 66.04 0)
 			(effects
 				(font
@@
 	(symbol
 		(lib_id "Device:R")
-		(at 154.94 54.61 0)
+		(at 152.4 60.96 0)
 		(mirror x)
 		(unit 1)
@@
 		(dnp no)
 		(property "Reference" "R8"
-			(at 152.4 53.3399 0)
+			(at 149.86 59.6899 0)
 			(effects
 				(font
@@
 		)
 		(property "Value" "4K7"
-			(at 152.4 55.8799 0)
+			(at 149.86 62.2299 0)
 			(effects
 				(font
@@
 		)
 		(property "Footprint" "Resistor_THT:R_Axial_DIN0207_L6.3mm_D2.5mm_P10.16mm_Horizontal"
-			(at 153.162 54.61 90)
+			(at 150.622 60.96 90)
 			(effects
 				(font
@@
 		)
 		(property "Datasheet" "~"
-			(at 154.94 54.61 0)
+			(at 152.4 60.96 0)
 			(effects
 				(font
@@
 		)
 		(property "Description" "Resistor"
-			(at 154.94 54.61 0)
+			(at 152.4 60.96 0)
 			(effects
 				(font
@@
 	(symbol
 		(lib_id "power:VCC")
-		(at 154.94 50.8 0)
+		(at 152.4 54.61 0)
 		(unit 1)
 		(exclude_from_sim no)
@@
 		(fields_autoplaced yes)
 		(property "Reference" "#PWR028"
-			(at 154.94 54.61 0)
+			(at 152.4 58.42 0)
 			(effects
 				(font
@@
 		)
 		(property "Value" "VCC"
-			(at 154.94 45.72 0)
+			(at 152.4 49.53 0)
 			(effects
 				(font
@@
 		)
 		(property "Footprint" ""
-			(at 154.94 50.8 0)
+			(at 152.4 54.61 0)
 			(effects
 				(font
@@
 		)
 		(property "Datasheet" ""
-			(at 154.94 50.8 0)
+			(at 152.4 54.61 0)
 			(effects
 				(font
@@
 		)
 		(property "Description" "Power symbol creates a global label with name \"VCC\""
-			(at 154.94 50.8 0)
+			(at 152.4 54.61 0)
 			(effects
 				(font

Commit message: pcb: silkscreen updates, minor routing updates
Connections:
- net AT_~{CE}: now also U10.4; no longer U10.5
- net ~{AT_ROM}: now also U10.5; no longer U10.4
Changed lines of the file:
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@@
 		(lib_id "74xx:74LS08")
 		(at 196.85 133.35 0)
+		(mirror x)
 		(unit 2)
 		(exclude_from_sim no)
@@
 		(on_board yes)
 		(dnp no)
-		(fields_autoplaced yes)
 		(property "Reference" "U10"
-			(at 196.8417 124.46 0)
+			(at 196.85 125.476 0)
 			(effects
 				(font
@@
 		)
 		(property "Value" "74LS08"
-			(at 196.8417 127 0)
+			(at 196.596 127.762 0)
 			(effects
 				(font
